File: pcb/booth fendi/booth fendi.kicad_sch (KiCad schematic)
At the start: 7 parts, among them J1 Conn_01x01_Female, J3 Conn_01x05_Female, J4 Conn_01x03_Female, J5 Conn_01x07_Female, J6 Conn_01x05_Female, J7 Conn_01x03

Commit message: traced no silkscreen
Parts:
- removed J1: Conn_01x01_Female, Connector_Wire:SolderWire-0.75sqmm_1x01_D1.25mm_OD2.3mm, symbol Connector:Conn_01x01_Female
Connections:
- no-connect marks 0 -> 15
Other:
- note added: "ETH Module"
- note added: "RS-232 TO TTL"
- note added: "Sens A"
- note added: "Sens B"
- note added: "StepDown"
- moved on the sheet: J6
